File: board/music-box.kicad_sch (KiCad schematic)
At the start: 22 parts, among them J1 SPEAKER, J2 MEM2061-01-188-00-A, J3 PWR, J4 BTN_PWR, J5 RFID, U1 MAX98357AETE+T, U2 SC0918

Commit message: fixed issue with board (rx / tx swap for the sd card)
Connections:
- net SD_RX renamed SD_MOSI
- net SD_MOSI: now also U2.15 (GP11); no longer U2.16 (GP12)
- net SD_TX renamed SD_MISO
- net SD_MISO: now also U2.16 (GP12); no longer U2.15 (GP11)
Changed lines of the file:
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@@
     (effects (font (size 5 5)) (justify left bottom))
   )
-  (label "SD_TX" (at 35.56 101.6 0) (fields_autoplaced)
+  (label "SD_MOSI" (at 35.56 101.6 0) (fields_autoplaced)
     (effects (font (size 1.27 1.27)) (justify left bottom))
   )
@@
     (effects (font (size 1.27 1.27)) (justify right bottom))
   )
-  (label "SD_RX" (at 280.67 201.93 0) (fields_autoplaced)
+  (label "SD_MOSI" (at 280.67 201.93 0) (fields_autoplaced)
     (effects (font (size 1.27 1.27)) (justify left bottom))
   )
@@
     (effects (font (size 1.27 1.27)) (justify left bottom))
   )
-  (label "SD_RX" (at 35.56 104.14 0) (fields_autoplaced)
+  (label "SD_MISO" (at 35.56 104.14 0) (fields_autoplaced)
     (effects (font (size 1.27 1.27)) (justify left bottom))
   )
@@
     (effects (font (size 1.27 1.27)) (justify right bottom))
   )
-  (label "SD_TX" (at 280.67 191.77 0) (fields_autoplaced)
+  (label "SD_MISO" (at 280.67 191.77 0) (fields_autoplaced)
     (effects (font (size 1.27 1.27)) (justify left bottom))
   )
